File: LABPSU/LABPSU_PWR_IN/PCB design/LABPSU_PWR_IN/LABPSU_PWR_IN.kicad_sch (KiCad schematic)
At the start: 10 parts, among them J1 Conn_01x02_Pin, J2 Conn_01x04_Pin, J3 Conn_01x10_Pin, T2 Transformer_1P_2S, T3 Transformer_1P_1S

Commit message: Add files via upload
Parts:
- F1, F2, F3, F4: Dist.partnumber (none) -> 100.238.32; Distributor (none) -> Hestore; LINK (none) -> https://www.hestore.hu/prod_10023832.html#; Manifacturer (none) -> RoHS
- T2: value Transformer_1P_2S -> BV EI 305 2056; Dist.partnumber (none) -> 100.387.00; Distriburor (none) -> Hestore; I szekunder (none) -> 167mA; LINK (none) -> https://www.hestore.hu/prod_10038700.html; Manifacturer (none) -> HAHN; Power (none) -> 3VA; V Primer  (none) -> 230 V AC; V Szekunder (none) -> 9 V
- T3: value Transformer_1P_1S -> EI38; Dist.partnumber (none) -> 100.258.55; Distributor (none) -> HESTORE; I  (none) -> 0,6A; LINK (none) -> https://www.hestore.hu/prod_10025855.html; Manifacturer  (none) -> INDEL; V primer (none) -> 230; V secunder (none) -> 6
